Commit message: urdf updated

File: spotmicro.urdf (robot description, URDF)
Before this commit: robot SpotMicroAI, 28 links, 27 joints
Links:
- added link board; collision box size=0.45 0.20 0.02; visual mesh filename=package://spotmicro_description/meshes/stl/CP_Snowboard.stl scale=.0005 .0005 .0005
Joints:
- added joint attach-board: type revolute, parent front_left_toe_link, child board, origin xyz=0 -0.01 0.015 rpy=0 0 0, axis 0 1 0, limit lower=-3.0 upper=3.0 effort=1000.0 velocity=0.5
- joint front_right_foot: limit lower=-2.59 upper=0.1 effort=1000.0 velocity=0.5 -> lower=-2.59 upper=2.0 effort=1000.0 velocity=0.5
- joint rear_right_foot: limit lower=-2.59 upper=0.1 effort=1000.0 velocity=0.5 -> lower=-2.59 upper=2.0 effort=1000.0 velocity=0.5

Commit message: up down

File: spotmicro.urdf (robot description, URDF)
Before this commit: robot SpotMicroAI, 29 links, 28 joints
Links:
- removed link base_horiz_d
- added link world_horiz_d
- added link world_vert_d
Joints:
- removed joint base_horiz
- added joint world_horiz: type prismatic, parent world, child world_horiz_d, origin xyz=0 0 0 rpy=0 0 0, axis 1 0 0, limit lower=-10 upper=10 effort=1000.0 velocity=0.5
- added joint world_vert: type prismatic, parent world_horiz_d, child world_vert_d, origin xyz=0 0 0 rpy=0 0 0, axis 0 0 1, limit lower=-10 upper=10 effort=1000.0 velocity=0.5
- joint base_vert: parent base_horiz_d -> world_vert_d

Commit message: Its Jover

File: spotmicro.urdf (robot description, URDF)
Before this commit: robot SpotMicroAI, 30 links, 29 joints
Links:
- added link world_y_d
- added link world_yaw_d
Joints:
- added joint world_y: type prismatic, parent world_vert_d, child world_y_d, origin xyz=0 0 0 rpy=0 0 0, axis 0 1 0, limit lower=-10 upper=10 effort=1000.0 velocity=0.5
- added joint world_yaw: type revolute, parent world_y_d, child world_yaw_d, origin xyz=0 0 0 rpy=0 0 0, axis 0 0 1, limit lower=-4 upper=4 effort=1000.0 velocity=0.5
- joint base_vert: parent world_vert_d -> world_yaw_d
